File: SAR_v1_5/shield_ard.brd (EAGLE design)
At the start: 79.5 x 76.1 mm, 14 parts

Commit message: many componentes were placed in other position on the board
Parts:
- removed RST_RPI: (no value), pinhead:2X10
- added JP2, JP5, JP6, JP7, JP8: (no value), SparkFun-Retired:1X02
- MOTOR_PASO: device pinhead:2X10 -> pinhead:2X05
- RTC: device pinhead:1X06 -> pinhead:1X06/90
- moved R2 69.9 mm to (3.75, 44.8), turned to 0 degrees
- moved LED2 66.3 mm to (3.62, 40.6), turned to 270 degrees
- moved CONECTOR_RBPI 57.7 mm to (26.9, 7.00)
- moved RTC 54.4 mm to (7.25, 57.5), turned to 270 degrees
- moved MOTOR_PASO 38.8 mm to (34.5, 23.1), flipped to the bottom
- moved JP1_LEVEL_L 33.5 mm to (23.1, 32.4), turned to 270 degrees
- moved JP2_LEVEL_H 20.9 mm to (12.6, 32.4), turned to 270 degrees
- moved JP1 13.4 mm to (50.6, 35.8)
- moved JP2_AN 13.1 mm to (2.37, 11.3)
- moved JP3 13.1 mm to (2.38, 29.1)
- moved JP4_SER 13.1 mm to (50.6, 13.9)
- moved R1 8.41 mm to (7.25, 13.6)
- moved LED1 8.15 mm to (7.12, 17.1)
Connections:
- new net N$6: JP6.2, MOTOR_PASO.4
- new net N$7: JP7.1, MOTOR_PASO.7
- net DIR: now also JP5.1, JP5.2
- net EN: now also JP2.1, JP2.2
- net GND: now also MOTOR_PASO.10, MOTOR_PASO.8; no longer MOTOR_PASO.17, MOTOR_PASO.18, MOTOR_PASO.20, RST_RPI.1, RST_RPI.17, RST_RPI.18, RST_RPI.20, RST_RPI.3
- net HV1_RST: no longer RST_RPI.4
- net HV_5V: no longer RST_RPI.2
- net SENSR: now also JP8.1, JP8.2, MOTOR_PASO.9; no longer MOTOR_PASO.19
- net SERVO: now also JP7.2; no longer RST_RPI.19
- net STEP: now also JP6.1; no longer MOTOR_PASO.4
Routing:
- net SERVO: track 109.8 -> 0.00 mm
- net HV1_RST: track 77.7 -> 0.00 mm, vias 2 -> 0
- net STEP: track 60.4 -> 0.00 mm
- net HV_5V: track 59.0 -> 0.00 mm, vias 1 -> 0
- net LV1: track 38.8 -> 0.00 mm
- net LV: track 27.0 -> 0.00 mm
- net VCC_RBPI: track 25.2 -> 0.00 mm, vias 1 -> 0
- net SCL: track 22.1 -> 0.00 mm
- net DIR: track 18.2 -> 0.00 mm
- net SDA: track 17.3 -> 0.00 mm
- net EN: track 16.1 -> 0.00 mm
- net SENSR: track 9.19 -> 0.00 mm
- net N$3: track 4.54 -> 0.00 mm
- net N$2: track 3.79 -> 0.00 mm
Other:
- board size 79.5 x 76.1 mm -> 232.6 x 85.5 mm

Commit message: cambios minimos
Parts:
- moved MOTOR_PASO 4.81 mm to (33.8, 27.9)
- moved CONECTOR_RBPI 0.25 mm to (26.9, 7.25)
Changed lines of the file:
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@@
 <wire x1="-0.25" y1="68.5" x2="-0.25" y2="2.5" width="0.2" layer="20"/>
 <rectangle x1="22.125" y1="37.375" x2="44.125" y2="77.375" layer="21" rot="R270"/>
+<rectangle x1="4" y1="3.125" x2="49" y2="11.125" layer="21"/>
+<rectangle x1="29.625" y1="12.375" x2="37.625" y2="44.375" layer="22"/>
 </plain>
 <attributes>
@@
 <attribute name="VALUE" x="9.415" y="40.065" size="1.27" layer="27" rot="R270"/>
 </element>
-<element name="CONECTOR_RBPI" library="pinhead" library_urn="urn:adsk.eagle:library:325" package="2X10" package3d_urn="urn:adsk.eagle:package:22405/2" value="" x="26.875" y="7" smashed="yes">
-<attribute name="NAME" x="14.175" y="2.425" size="1.016" layer="25" font="vector" ratio="10"/>
-<attribute name="POPULARITY" value="7" x="26.875" y="7" size="1.778" layer="27" display="off"/>
-<attribute name="VALUE" x="14.175" y="2.555" size="1.27" layer="27"/>
+<element name="CONECTOR_RBPI" library="pinhead" library_urn="urn:adsk.eagle:library:325" package="2X10" package3d_urn="urn:adsk.eagle:package:22405/2" value="" x="26.875" y="7.25" smashed="yes">
+<attribute name="NAME" x="14.175" y="2.675" size="1.016" layer="25" font="vector" ratio="10"/>
+<attribute name="POPULARITY" value="7" x="26.875" y="7.25" size="1.778" layer="27" display="off"/>
+<attribute name="VALUE" x="14.175" y="2.805" size="1.27" layer="27"/>
 </element>
 <element name="LED1" library="led" library_urn="urn:adsk.eagle:library:259" package="CHIP-LED0805" package3d_urn="urn:adsk.eagle:package:15818/2" value="" x="7.125" y="17.125" smashed="yes" rot="R270">
@@
 <attribute name="VALUE" x="40.98" y="16.093" size="0.6096" layer="27" font="vector" ratio="20"/>
 </element>
-<element name="MOTOR_PASO" library="pinhead" library_urn="urn:adsk.eagle:library:325" package="2X05" package3d_urn="urn:adsk.eagle:package:22470/2" value="" x="34.5" y="23.125" smashed="yes" rot="MR270">
-<attribute name="NAME" x="31.325" y="29.475" size="1.27" layer="26" ratio="10" rot="MR270"/>
-<attribute name="POPULARITY" value="35" x="34.5" y="23.125" size="1.778" layer="28" rot="MR270" display="off"/>
-<attribute name="VALUE" x="38.945" y="29.475" size="1.27" layer="28" rot="MR270"/>
+<element name="MOTOR_PASO" library="pinhead" library_urn="urn:adsk.eagle:library:325" package="2X05" package3d_urn="urn:adsk.eagle:package:22470/2" value="" x="33.75" y="27.875" smashed="yes" rot="MR270">
+<attribute name="NAME" x="30.575" y="34.225" size="1.27" layer="26" ratio="10" rot="MR270"/>
+<attribute name="POPULARITY" value="35" x="33.75" y="27.875" size="1.778" layer="28" rot="MR270" display="off"/>
+<attribute name="VALUE" x="38.195" y="34.225" size="1.27" layer="28" rot="MR270"/>
 </element>
 <element name="RTC" library="pinhead" library_urn="urn:adsk.eagle:library:325" package="1X06/90" package3d_urn="urn:adsk.eagle:package:22475/2" value="" x="7.25" y="57.5" smashed="yes" rot="R270">
@@
 <contactref element="MOTOR_PASO" pad="2"/>
 <contactref element="RTC" pad="1"/>
-<wire x1="33.225" y1="5.73" x2="50.625" y2="42.1" width="0" layer="19" extent="1-1"/>
-<wire x1="28.145" y1="8.27" x2="33.225" y2="5.73" width="0" layer="19" extent="1-1"/>
-<wire x1="6.3" y1="13.625" x2="28.145" y2="8.27" width="0" layer="19" extent="1-1"/>
+<wire x1="33.225" y1="5.98" x2="50.625" y2="42.1" width="0" layer="19" extent="1-1"/>
+<wire x1="28.145" y1="8.52" x2="33.225" y2="5.98" width="0" layer="19" extent="1-1"/>
+<wire x1="6.3" y1="13.625" x2="28.145" y2="8.52" width="0" layer="19" extent="1-1"/>
 <wire x1="2.375" y1="25.315" x2="6.3" y2="13.625" width="0" layer="19" extent="1-1"/>
 <wire x1="2.375" y1="27.855" x2="2.375" y2="25.315" width="0" layer="19" extent="1-1"/>
 <wire x1="2.8" y1="44.75" x2="2.375" y2="27.855" width="0" layer="19" extent="1-1"/>
-<wire x1="33.23" y1="18.045" x2="2.375" y2="27.855" width="0" layer="19" extent="1-1"/>
-<wire x1="33.23" y1="20.585" x2="33.23" y2="18.045" width="0" layer="19" extent="1-1"/>
-<wire x1="33.23" y1="28.205" x2="33.23" y2="20.585" width="0" layer="19" extent="1-1"/>
+<wire x1="32.48" y1="22.795" x2="2.375" y2="27.855" width="0" layer="19" extent="1-1"/>
+<wire x1="32.48" y1="25.335" x2="32.48" y2="22.795" width="0" layer="19" extent="1-1"/>
+<wire x1="32.48" y1="32.955" x2="32.48" y2="25.335" width="0" layer="19" extent="1-1"/>
 <wire x1="3.44" y1="63.85" x2="2.8" y2="44.75" width="0" layer="19" extent="1-1"/>
-<wire x1="12.59" y1="33.715" x2="33.23" y2="28.205" width="0" layer="19" extent="1-1"/>
+<wire x1="12.59" y1="33.715" x2="32.48" y2="32.955" width="0" layer="19" extent="1-1"/>
 <wire x1="23.06" y1="31.175" x2="12.59" y2="33.715" width="0" layer="19" extent="1-1"/>
 </signal>
@@
 <wire x1="44.415" y1="26.875" x2="50.625" y2="26.86" width="0" layer="19" extent="1-1"/>
 <wire x1="41.875" y1="26.875" x2="44.415" y2="26.875" width="0" layer="19" extent="1-1"/>
-<wire x1="35.77" y1="28.205" x2="41.875" y2="26.875" width="0" layer="19" extent="1-1"/>
+<wire x1="35.02" y1="32.955" x2="41.875" y2="26.875" width="0" layer="19" extent="1-1"/>
 </signal>
 <signal name="DIR">
@@
 <wire x1="44.665" y1="22.5" x2="50.625" y2="22.775" width="0" layer="19" extent="1-1"/>
 <wire x1="42.125" y1="22.5" x2="44.665" y2="22.5" width="0" layer="19" extent="1-1"/>
-<wire x1="35.77" y1="25.665" x2="42.125" y2="22.5" width="0" layer="19" extent="1-1"/>
+<wire x1="35.02" y1="30.415" x2="42.125" y2="22.5" width="0" layer="19" extent="1-1"/>
 </signal>
 <signal name="STEP">
@@
 <wire x1="44.79" y1="18.125" x2="50.625" y2="17.695" width="0" layer="19" extent="1-1"/>
 <wire x1="42.25" y1="18.125" x2="44.79" y2="18.125" width="0" layer="19" extent="1-1"/>
-<wire x1="35.77" y1="18.045" x2="42.25" y2="18.125" width="0" layer="19" extent="1-1"/>
+<wire x1="35.02" y1="22.795" x2="42.25" y2="18.125" width="0" layer="19" extent="1-1"/>
 </signal>
 <signal name="LV1">
 <contactref element="JP1_LEVEL_L" pad="1"/>
 <contactref element="CONECTOR_RBPI" pad="6"/>
-<wire x1="20.525" y1="8.27" x2="23.06" y2="38.795" width="0" layer="19" extent="1-1"/>
+<wire x1="20.525" y1="8.52" x2="23.06" y2="38.795" width="0" layer="19" extent="1-1"/>
 </signal>
 <signal name="LV2">
@@
 <contactref element="JP1_LEVEL_L" pad="3"/>
 <contactref element="CONECTOR_RBPI" pad="4"/>
-<wire x1="17.985" y1="8.27" x2="23.06" y2="33.715" width="0" layer="19" extent="1-1"/>
+<wire x1="17.985" y1="8.52" x2="23.06" y2="33.715" width="0" layer="19" extent="1-1"/>
 </signal>
 <signal name="LV3">
@@
 <contactref element="RTC" pad="2"/>
 <wire x1="2.575" y1="40.625" x2="3.44" y2="61.31" width="0" layer="19" extent="1-1"/>
-<wire x1="38.305" y1="8.27" x2="2.575" y2="40.625" width="0" layer="19" extent="1-1"/>
+<wire x1="38.305" y1="8.52" x2="2.575" y2="40.625" width="0" layer="19" extent="1-1"/>
 </signal>
 <signal name="SDA">
 <contactref element="CONECTOR_RBPI" pad="18"/>
 <contactref element="RTC" pad="3"/>
-<wire x1="35.765" y1="8.27" x2="3.44" y2="58.77" width="0" layer="19" extent="1-1"/>
+<wire x1="35.765" y1="8.52" x2="3.44" y2="58.77" width="0" layer="19" extent="1-1"/>
 </signal>
 <signal name="SCL">
 <contactref element="CONECTOR_RBPI" pad="16"/>
 <contactref element="RTC" pad="4"/>
-<wire x1="33.225" y1="8.27" x2="3.44" y2="56.23" width="0" layer="19" extent="1-1"/>
+<wire x1="33.225" y1="8.52" x2="3.44" y2="56.23" width="0" layer="19" extent="1-1"/>
 </signal>
 <signal name="HV1_RST">
@@
 <contactref element="JP6" pad="2"/>
 <contactref element="MOTOR_PASO" pad="4"/>
-<wire x1="33.23" y1="25.665" x2="41.71" y2="31.625" width="0" layer="19" extent="1-1"/>
+<wire x1="32.48" y1="30.415" x2="41.71" y2="31.625" width="0" layer="19" extent="1-1"/>
 </signal>
 <signal name="N$7">
 <contactref element="JP7" pad="1"/>
 <contactref element="MOTOR_PASO" pad="7"/>
-<wire x1="35.77" y1="20.585" x2="44.875" y2="13.875" width="0" layer="19" extent="1-1"/>
+<wire x1="35.02" y1="25.335" x2="44.875" y2="13.875" width="0" layer="19" extent="1-1"/>
 </signal>
 <signal name="N$41">
